Commit message: modified urdf and added planner pkg

File: robot_description/urdf/gripper1.urdf (robot description, URDF)
Before this commit: robot gripper_v1, 7 links, 6 joints
Links:
- added link link_10, mass 1.0; collision box size=0.1 0.7 0.2; visual box size=0.1 0.7 0.2
- added link link_11, mass 1.0; collision cylinder length=0.2 radius=0.05; visual cylinder length=0.2 radius=0.05
- added link link_12, mass 1.0; collision cylinder length=0.2 radius=0.05; visual cylinder length=0.2 radius=0.05
- added link link_13, mass 1.0; collision box size=0.1 0.5 0.2; visual box size=0.1 0.5 0.2
- added link link_14, mass 1.0; collision box size=0.1 0.5 0.2; visual box size=0.1 0.5 0.2
- added link link_15, mass 1.0; collision sphere radius=0.1; visual sphere radius=0.1
- added link link_16, mass 1.0; collision sphere radius=0.1; visual sphere radius=0.1
- added link link_7, mass 1.0; collision cylinder length=0.2 radius=0.05; visual cylinder length=0.2 radius=0.05
- added link link_8, mass 1.0; collision cylinder length=0.2 radius=0.05; visual cylinder length=0.2 radius=0.05
- added link link_9, mass 1.0; collision box size=0.1 0.7 0.2; visual box size=0.1 0.7 0.2
- added link map
- link link_2: geometry collision box size=0.3 0.2 0.2; visual box size=0.3 0.2 0.2
- link link_3: geometry collision cylinder length=0.2 radius=0.05; visual cylinder length=0.2 radius=0.05
- link link_4: geometry collision cylinder length=0.2 radius=0.05; visual cylinder length=0.2 radius=0.05
- link link_5: geometry collision box size=0.2 0.2 0.1; visual box size=0.2 0.2 0.1
- link link_6: geometry collision box size=0.2 0.2 0.1; visual box size=0.2 0.2 0.1
Joints:
- added joint joint_0: type fixed, parent map, child base_link, origin xyz=0 0 0.025 rpy=0 0 0
- added joint joint_10: type fixed, parent link_8, child link_10, origin xyz=0 0.4 0 rpy=0 0 0
- added joint joint_11: type revolute, parent link_9, child link_11, origin xyz=0 0.4 0 rpy=0 0 1.04, axis 0 0 1, limit lower=-1.57 upper=1.57 effort=10 velocity=5
- added joint joint_12: type revolute, parent link_10, child link_12, origin xyz=0 0.4 0 rpy=0 0 -1.04, axis 0 0 1, limit lower=-1.57 upper=1.57 effort=10 velocity=5
- added joint joint_13: type fixed, parent link_11, child link_13, origin xyz=0 0.3 0 rpy=0 0 0
- added joint joint_14: type fixed, parent link_12, child link_14, origin xyz=0 0.3 0 rpy=0 0 0
- added joint joint_15: type fixed, parent link_13, child link_15, origin xyz=0 0.35 0 rpy=0 0 0
- added joint joint_16: type fixed, parent link_14, child link_16, origin xyz=0 0.35 0 rpy=0 0 0
- added joint joint_7: type revolute, parent link_5, child link_7, origin xyz=0.15 0 0 rpy=1.57 0.26 0, axis 0 0 1, limit lower=-1.57 upper=1.57 effort=10 velocity=5
- added joint joint_8: type revolute, parent link_6, child link_8, origin xyz=-0.15 0 0 rpy=1.57 -0.26 0, axis 0 0 1, limit lower=-1.57 upper=1.57 effort=10 velocity=5
- added joint joint_9: type fixed, parent link_7, child link_9, origin xyz=0 0.4 0 rpy=0 0 0
- joint joint_1: axis 0 1 0 -> (none); limit lower=-1.57 upper=1.57 effort=10 velocity=5 -> (none); type revolute -> fixed
- joint joint_3: axis 0 1 0 -> 0 0 1; origin xyz=0.5 0 0.2 rpy=0 0.785 0 -> xyz=0.2 0 0 rpy=0 0 0
- joint joint_4: axis 0 1 0 -> 0 0 1; origin xyz=-0.5 0 0.2 rpy=0 -0.785 0 -> xyz=-0.2 0 0 rpy=0 0 0
- joint joint_5: axis 0 1 0 -> (none); limit lower=-1.57 upper=1.57 effort=10 velocity=5 -> (none); origin xyz=0.5 0 0.2 rpy=0 0.785 0 -> xyz=0.15 0 0 rpy=0 0 0; type revolute -> fixed
- joint joint_6: axis 0 1 0 -> (none); limit lower=-1.57 upper=1.57 effort=10 velocity=5 -> (none); origin xyz=-0.5 0 0.2 rpy=0 -0.785 0 -> xyz=-0.15 0 0 rpy=0 0 0; type revolute -> fixed

Commit message: moveit package created

File: robot_description/urdf/gripper1.urdf (robot description, URDF)
Before this commit: robot gripper_v1, 18 links, 17 joints
Joints:
- joint joint_2: axis (none) -> 0 0 1; limit (none) -> lower=-1.57 upper=1.57 effort=10 velocity=5; type fixed -> revolute
